File: PCB/MarvinPeripheralsDeck.kicad_sch (KiCad schematic)
At the start: 18 parts, among them SW2 SW_Push, SW3 SW_Push, U2 BMP280, U3 LSM6DSOTR, U4 LIS3MDLTR, U5 MS5611-01BA

Commit message: v2!
Parts:
- removed JP3, JP6: SB C, Jumper:SolderJumper-2_P1.3mm_Bridged_Pad1.0x1.5mm, symbol Jumper:SolderJumper_2_Bridged
- removed JP4, JP5: SB O, Jumper:SolderJumper-2_P1.3mm_Open_Pad1.0x1.5mm, symbol Jumper:SolderJumper_2_Open
- added BZ1: Buzzer, Buzzer_Beeper:Buzzer_12x9.5RM7.6, symbol Device:Buzzer
- added Q5: BC847, Package_TO_SOT_SMD:SOT-23, symbol Transistor_BJT:BC847
- added R47: 1k, Resistor_SMD:R_0603_1608Metric, symbol Device:R
Connections:
- net GND: now also U3.1 (SDO/SA0), U4.9 (SDO/SA1), U5.4 (CSB), U5.5 (CSB), Q5.2 (E)
- net IMU.SCL: now also U4.1 (SCL/SPC)
- net IMU.SDA: now also U4.11 (SDA/SDI/SDO)
- new net: Q5.1 (B), R47.1
- new net: BZ1.2 (+), Q5.3 (C)
- new net +5VP: BZ1.1 (-)
- new net BUZZER: R47.2
- no-connect marks 7 -> 4
Other:
- note added: "LSM6DSO is the master of LIS3MDL over the I2CF(usion) bus, no pullups needed, DRDY is a data ready interrupt for I2C sync between the sensors"
- note removed: "LSM6DSO is a master of LIS3MDL over the I2CF(usion) bus, no pullups needed, DRDY is a data ready interrupt for I2C sync between the sensors"
- moved on the sheet: C14, C15, R7, R8, SW2, SW3
