File: PCB/comms.kicad_sch (KiCad schematic)
At the start: 8 parts, among them J16 MEM2051-00-195-00-A, U11 W25Q16JLSSIG, U12 RA-02_LORA

Commit message: v2!
Parts:
- removed J16: MEM2051-00-195-00-A, SD:MEM2051-00-195-00-A, symbol MEM:MEM2051-00-195-00-A
- added K1: 112J-TDAR-R01, newsd:112J-TDAR-R01, symbol newsd:112J-TDAR-R01
Connections:
- net +3V3: now also K1.4 (4-VDD)
- net GND: now also K1.6 (6-VSS)
- net TF.MISO: now also K1.7 (7-DAT0)
- net TF.MOSI: now also K1.3 (3-CMD)
- net TF.SCK: now also K1.5 (5-CLK)
- net at JP7.1 (A): now also K1.2 (2-CD/DAT3)
