File: PCB/marvin_fc_board.kicad_pcb (KiCad board)
At the start: 4 copper layers, 65 x 100 mm, 164 parts, among them J1 PROG / DBG, J10 EXP1, J11 EXP2, J12 POWER_IN, J13 EXTl NTC, J14 Screw_Terminal_01x05, J15 ATTINY_DBG, J16 MEM2051-00-195-00-A, J17 Pyro Terminal 1, J18 Pyro Terminal 2, J2 EXPA, J3 EXPC, J4 SERVO POW 1, J5 SERVO POW 2, J6 EXPB, J7 EXPD, J8 SERVO SIG 1, J9 SERVO SIG 2, Q1 SISH101DN, Q2 SISH101DN, Q3 BC847, Q4 AO4822A, SW1 SW_Push, SW2 SW_Push, SW3 SW_Push, U1 STM32F407, U10 TXB0108DQSR, U11 W25Q16JLSSIG, U12 RA-02_LORA, U13 ILD213T, U14 AP62200Z6, U15 AP62200Z6, U16 MCP9700AT-ELT, U17 MCP9700AT-ELT, U18 MCP9700AT-ELT, U2 BMP280, U3 LSM6DSOTR, U4 LIS3MDLTR, U5 MS5611-01BA, U6 NCP718xSN500, U7 ST1S41PHR, U8 PAC1954, U9 ATtiny1627-M, Y1 Crystal_GND24

Commit message: v2!
Parts:
- removed D1: LED_RGBK, LED_SMD:LED_Cree-PLCC4_2x2mm_CW
- removed J16: MEM2051-00-195-00-A, SD:MEM2051-00-195-00-A
- removed JP3, JP6: SB C, Jumper:SolderJumper-2_P1.3mm_Bridged_Pad1.0x1.5mm
- removed JP4, JP5: SB O, Jumper:SolderJumper-2_P1.3mm_Open_Pad1.0x1.5mm
- removed the REF** at (155.4, 150.8)
- removed the REF** at (155.3, 57.0)
- removed the REF** at (96.5, 57.0)
- removed the REF** at (96.6, 150.9)
- added ?: , , F.Cu at (155.3, 57.2)
- added ?: , , F.Cu at (96.7, 57.2)
- added ?: , , F.Cu at (155.3, 150.8)
- added BZ1: Buzzer, Buzzer_Beeper:Buzzer_12x9.5RM7.6, B.Cu at (136.1, 110.3)
- added D8: LED_RGBA, LED_SMD:LED_Cree-PLCC4_2x2mm_CW, F.Cu at (109.3, 88.2)
- added F3: 200mA, Fuse:Fuse_0603_1608Metric, F.Cu at (149.0, 65.2)
- added J19: SERVO4 PINS, Connector_PinHeader_2.54mm:PinHeader_1x03_P2.54mm_Vertical, F.Cu at (107.7, 58.4)
- added J20: SERVO5 PINS, Connector_PinHeader_2.54mm:PinHeader_1x03_P2.54mm_Vertical, F.Cu at (107.7, 55.8)
- added J22: EXT_PWR, Connector_PinHeader_2.54mm:PinHeader_1x03_P2.54mm_Vertical, F.Cu at (153.0, 62.4)
- added J23: EXT_GND, Connector_PinHeader_2.54mm:PinHeader_1x03_P2.54mm_Vertical, F.Cu at (155.8, 62.4)
- added K1: 112J-TDAR-R01, newsd:112J-TDAR-R01, B.Cu at (103.8, 108.9)
- added Q5: BC847, Package_TO_SOT_SMD:SOT-23, B.Cu at (146.9, 98.6)
- added R47: 1k, Resistor_SMD:R_0603_1608Metric, B.Cu at (147.0, 95.3)
- added REF**: MountingHole_3.2mm_M3_ISO7380_Pad, MountingHole:MountingHole_3.2mm_M3_ISO7380_Pad, F.Cu at (96.7, 150.8)
- added TP4: TestPoint, TestPoint:TestPoint_Pad_D1.0mm, F.Cu at (136.0, 78.0)
- added kibuzzard-63A8BFA0: G***, kibuzzard-63A8BFA0, F.Cu at (102.4, 48.8)
- added kibuzzard-63A8DA8E: G***, kibuzzard-63A8DA8E, F.Cu at (122.5, 50.7)
- added kibuzzard-63A8DDC0: G***, kibuzzard-63A8DDC0, F.Cu at (102.6, 63.1)
- added kibuzzard-63A8DDCD: G***, kibuzzard-63A8DDCD, F.Cu at (105.1, 63.1)
- added kibuzzard-63A8DDD8: G***, kibuzzard-63A8DDD8, F.Cu at (107.7, 63.1)
- added kibuzzard-63A8E0B0: G***, kibuzzard-63A8E0B0, F.Cu at (111.3, 61.7)
- added kibuzzard-63A8E0BF: G***, kibuzzard-63A8E0BF, F.Cu at (111.3, 59.0)
- added kibuzzard-63A8E0CA: G***, kibuzzard-63A8E0CA, F.Cu at (111.2, 56.3)
- added kibuzzard-63A8E131: G***, kibuzzard-63A8E131, F.Cu at (128.4, 56.4)
- added kibuzzard-63A8E13C: G***, kibuzzard-63A8E13C, F.Cu at (128.4, 59.0)
- added kibuzzard-63A8E14B: G***, kibuzzard-63A8E14B, F.Cu at (96.6, 71.2)
- added kibuzzard-63A8E197: G***, kibuzzard-63A8E197, F.Cu at (157.8, 70.6)
- added kibuzzard-63A8E1B3: G***, kibuzzard-63A8E1B3, F.Cu at (146.7, 114.7)
- added kibuzzard-63A8E1B7: G***, kibuzzard-63A8E1B7, F.Cu at (146.7, 121.4)
- added kibuzzard-63A8E1BC: G***, kibuzzard-63A8E1BC, F.Cu at (146.8, 127.7)
- added kibuzzard-63A8E1E9: G***, kibuzzard-63A8E1E9, F.Cu at (155.0, 143.4)
- added kibuzzard-63A8E1FE: G***, kibuzzard-63A8E1FE, F.Cu at (95.1, 115.2)
- added kibuzzard-63A8E239: G***, kibuzzard-63A8E239, F.Cu at (95.1, 123.0)
- added kibuzzard-63A8E3F2: G***, kibuzzard-63A8E3F2, F.Cu at (105.8, 146.1)
- added kibuzzard-63AA0089: G***, kibuzzard-63AA0089, F.Cu at (98.6, 98.7)
- added kibuzzard-63AA01CF: G***, kibuzzard-63AA01CF, F.Cu at (177.5, 78.5)
- added kibuzzard-63AA020A: G***, kibuzzard-63AA020A, F.Cu at (48.5, 127.7)
- added kibuzzard-63AA024E: G***, kibuzzard-63AA024E, F.Cu at (99.7, 93.5)
- added kibuzzard-63AA0256: G***, kibuzzard-63AA0256, F.Cu at (99.6, 90.9)
- added kibuzzard-63AA025D: G***, kibuzzard-63AA025D, F.Cu at (100.7, 88.3)
- added kibuzzard-63AA0264: G***, kibuzzard-63AA0264, F.Cu at (100.5, 85.7)
- added kibuzzard-63AA0274: G***, kibuzzard-63AA0274, F.Cu at (99.0, 83.2)
- added kibuzzard-63AA02A3: G***, kibuzzard-63AA02A3, F.Cu at (96.2, 75.8)
- added kibuzzard-63AA02B1: G***, kibuzzard-63AA02B1, F.Cu at (98.8, 75.8)
- added kibuzzard-63AA0354: G***, kibuzzard-63AA0354, F.Cu at (101.3, 75.8)
- added kibuzzard-63AC1524: G***, kibuzzard-63AC1524, F.Cu at (99.2, 78.2)
- added kibuzzard-63AC1538: G***, kibuzzard-63AC1538, F.Cu at (101.4, 80.5)
- added kibuzzard-63AC1541: G***, kibuzzard-63AC1541, F.Cu at (102.1, 77.5)
- C38, C39: value 100u -> 10u
- J2: value EXPA -> OUT_A
- J3: value EXPC -> OUT_C
- J4: value SERVO POW 1 -> SERVO0 JST; footprint Connector_PinHeader_2.54mm:PinHeader_2x03_P2.54mm_Vertical -> Connector_JST:JST_XH_B3B-XH-A_1x03_P2.50mm_Vertical
- J5: value SERVO POW 2 -> SERVO1 JST; footprint Connector_PinHeader_2.54mm:PinHeader_2x03_P2.54mm_Vertical -> Connector_JST:JST_XH_B3B-XH-A_1x03_P2.50mm_Vertical
- J6: value EXPB -> OUT_B
- J7: value EXPD -> OUT_D
- J8: value SERVO SIG 1 -> SERVO2 JST; footprint Connector_PinHeader_2.54mm:PinHeader_1x03_P2.54mm_Vertical -> Connector_JST:JST_XH_B3B-XH-A_1x03_P2.50mm_Vertical
- J9: value SERVO SIG 2 -> SERVO3 PINS
- Q4: value AO4822A -> DMN3018SSD
- R1: value 510ohm -> 1k
- R10, R14: value 2137 -> 56k
- R11: value 42069 -> 10k
- R12: value ? -> 330k
- R13: value ? -> 100k
- R15: value R -> 10k
- R27, R29, R30, R31: value R -> 500
- TP3: moved to B.Cu
- U6: value NCP718xSN500 -> LM1117-5.0; footprint Package_TO_SOT_SMD:SOT-23-5 -> Package_TO_SOT_SMD:SOT-223-3_TabPin2
- U8: footprint Package_DFN_QFN:UQFN-16-1EP_4x4mm_P0.65mm_EP2.7x2.7mm -> Package_DFN_QFN:VQFN-16-1EP_3x3mm_P0.5mm_EP1.1x1.1mm
- moved J5 74.7 mm to (150.1, 119.9), turned to 0 degrees
- moved TP2 39.4 mm to (134.7, 147.4)
- moved J8 34.1 mm to (150.1, 113.4), turned to 0 degrees
- moved J4 26.4 mm to (150.1, 126.4), turned to 0 degrees
- moved C28 12.0 mm to (99.4, 146.1), turned to 180 degrees
- moved C34 10.7 mm to (117.2, 105.7), turned to -90 degrees
- moved JP7 6.27 mm to (120.0, 104.3), turned to -90 degrees
- moved JP1 5.78 mm to (115.3, 94.8), turned to 180 degrees
- moved R23 3.67 mm to (152.2, 142.8)
- moved D3 3.56 mm to (152.2, 139.1)
- moved D4 3.56 mm to (152.3, 128.8)
- moved R27 3.56 mm to (152.2, 140.9)
- moved R30 3.56 mm to (152.2, 134.0)
- moved R29 3.56 mm to (152.2, 130.5)
- moved D5 3.56 mm to (152.2, 132.2)
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Connections:
- net /EXP1 renamed /GPIO1
- net /EXP2 renamed /GPIO2
- net /PORTA0 renamed /PD0
- net /PORTA1 renamed /PD1
- net /PORTA10 renamed /PD10
- net /PORTA11 renamed /PD11
- net /PORTA12 renamed /PD12
- net /PORTA13 renamed /PD13
- net /PORTA14 renamed /PD14
- net /PORTA15 renamed /PD15
- net /PORTA2 renamed /PD2
- net /PORTA3 renamed /PD3
- net /PORTA4 renamed /PD4
- net /PORTA5 renamed /PD5
- net /PORTA6 renamed /PD6
- net /PORTA7 renamed /PD7
- net /PORTA8 renamed /PD8
- net /PORTA9 renamed /PD9
- C17 pad 1: Net-(C17-Pad1) -> Net-(D2-A)
- D2 pad 2: Net-(C17-Pad1) -> Net-(D2-A)
- J4 pad 1: GND -> /PWM0
- J5 pad 1: GND -> /PWM1
- J8 pad 1: /PWM0 -> /PWM2
- J8 pad 2: /PWM1 -> +5VP
- J8 pad 3: /PWM2 -> GND
- J9 pad 1: /PWM5 -> /PWM3
- J9 pad 2: /PWM4 -> +5VP
- J9 pad 3: /PWM3 -> GND
- R5 pad 2: GND -> +3V3
- U1 pad 37: unconnected-(U1-Pad37) -> Net-(U1-PB2)
- U1 pad 92: /DBG_UART_RX -> /DBG_UART_TX
- U1 pad 93: /DBG_UART_TX -> /DBG_UART_RX
- U10 pad 1: unconnected-(U10-Pad1) -> GND
- U10 pad 14: unconnected-(U10-Pad14) -> GND
- U10 pad 15: unconnected-(U10-Pad15) -> GND
- U10 pad 20: unconnected-(U10-Pad20) -> GND
- U10 pad 6: unconnected-(U10-Pad6) -> GND
- U10 pad 7: unconnected-(U10-Pad7) -> GND
- U3 pad 1: unconnected-(U3-Pad1) -> GND
- U4 pad 1: Net-(JP3-Pad2) -> /I2C2.SCL
- U4 pad 11: Net-(JP5-Pad2) -> /I2C2.SDA
- U4 pad 9: unconnected-(U4-Pad9) -> GND
- U5 pad 4: unconnected-(U5-Pad4) -> GND
- U5 pad 5: unconnected-(U5-Pad4) -> GND
- U6 pad 1: VBUS -> GND
- U6 pad 2: GND -> Net-(D2-A)
Routing:
- net +5VP: track 198.8 -> 275.6 mm, vias 6 -> 7
- net /PWM2: track 89.0 -> 60.4 mm
- net /PWM1: track 89.1 -> 64.1 mm
- net VBUS: track 45.6 -> 26.0 mm
- net /PD12: track 44.6 -> 63.3 mm
- net /PWM0: track 89.9 -> 71.6 mm
- net /Marvin Peripherals Deck/I2CF_SDA: track 13.4 -> 0.00 mm, vias 1 -> 0
- net Net-(D2-A): track 0.00 -> 13.0 mm
- net Net-(BZ1-+): track 0.00 -> 13.0 mm
- net GND: track 58.9 -> 67.6 mm
- net Net-(C17-Pad1): track 6.72 -> 0.00 mm
- net /TF_CS: track 55.2 -> 48.7 mm
- net /PWM5: track 35.7 -> 42.1 mm
- net Net-(U1-PB2): track 0.00 -> 6.24 mm
- net /IMU_INT: track 31.6 -> 25.5 mm
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Other:
- outline, holes or cut-outs redrawn
- board text added: "PWR"
- board text removed: "EXP1"
- board text removed: "EXP2"
- board text removed: "F"
- board text removed: "MAG_SCL"
- board text removed: "MAG_SDA"
- board text removed: "RX"
- board text removed: "SWCLK"
- board text removed: "SWDIO"
