File: PCB/marvin_fc_board.kicad_sch (KiCad schematic)
At the start: 22 parts, among them SW1 SW_Push, U1 STM32F407, Y1 Crystal_GND24

Commit message: v2!
Parts:
- removed D1: LED_RGBK, LED_SMD:LED_Cree-PLCC4_2x2mm_CW, symbol Device:LED_RGBK
- added D8: LED_RGBA, LED_SMD:LED_Cree-PLCC4_2x2mm_CW, symbol Device:LED_RGBA
- added TP4: TestPoint, TestPoint:TestPoint_Pad_D1.0mm, symbol Connector:TestPoint
- R1: value 510ohm -> 1k
Connections:
- net +3V3: now also R5.2
- net B: now also D8.3 (BK)
- net DBG_UART_RX: now also U1.93 (PB7); no longer U1.92 (PB6)
- net DBG_UART_TX: now also U1.92 (PB6); no longer U1.93 (PB7)
- net G: now also D8.2 (GK)
- net GND: no longer R5.2
- net R: now also D8.1 (RK)
- net at R5.1: now also D8.4 (A)
- net at U1.37 (PB2): now also TP4.1
- net EXP1 renamed GPIO1
- net EXP2 renamed GPIO2
- net PORTA0 renamed PD0
- net PORTA1 renamed PD1
- net PORTA10 renamed PD10
- net PORTA11 renamed PD11
- net PORTA12 renamed BUZZER_PWM
- net PORTA13 renamed PD13
- net PORTA14 renamed PD14
- net PORTA15 renamed PD15
- net PORTA2 renamed PD2
- net PORTA3 renamed PD3
- net PORTA4 renamed PD4
- net PORTA5 renamed PD5
- net PORTA6 renamed PD6
- net PORTA7 renamed PD7
- net PORTA8 renamed PD8
- net PORTA9 renamed PD9
Other:
- sheet Marvin Peripherals Deck ports: added BUZZER; removed none
