File: PCB/psu_board.kicad_sch (KiCad schematic)
At the start: 60 parts, among them J12 POWER_IN, J13 EXTl NTC, J14 Screw_Terminal_01x05, J15 ATTINY_DBG, Q1 SISH101DN, Q2 SISH101DN, Q3 BC847, U10 TXB0108DQSR, U6 NCP718xSN500, U7 ST1S41PHR, U8 PAC1954, U9 ATtiny1627-M

Commit message: v2!
Parts:
- removed U6: NCP718xSN500, Package_TO_SOT_SMD:SOT-23-5, symbol Regulator_Linear:NCP718xSN500
- added U6: LM1117-5.0, Package_TO_SOT_SMD:SOT-223-3_TabPin2, symbol Regulator_Linear:LM1117-5.0
- R10, R14: value 2137 -> 56k
- R11: value 42069 -> 10k
- R12: value ? -> 330k
- R13: value ? -> 100k
- R15: value R -> 10k
- U8: footprint Package_DFN_QFN:UQFN-16-1EP_4x4mm_P0.65mm_EP2.7x2.7mm -> Package_DFN_QFN:VQFN-16-1EP_3x3mm_P0.5mm_EP1.1x1.1mm
Connections:
- net GND: now also U10.1 (A1), U10.14 (B6), U10.15 (B5), U10.20 (B1), U10.6 (A5), U10.7 (A6), U6.1 (GND)
- net VBUS: now also U6.3 (VI)
- net at C17.1, D2.2 (A): now also U6.2 (VO)
Other:
- note added: "Power Supply Section Generates 3.3V, 5V for logic, 5V for Expansion and Unregulated Four rails are independentily monitored Also provides 3 temperature sensors Attiny communictes with the main system processor over SPI"
- note added: "Vout: 3.3V"
- note added: "Vout: 5,28V"
- note added: "Vout: 5V"
- note removed: "Power Supply Section Generates 3.3V, 5V for logic, 5V for Expansion and Unregulated Four rail are independentily monitored Also provides 3 temperature sensors Attiny communictes with the main system processor over SPI"
