File: PCB/pyro_sheet.kicad_sch (KiCad schematic)
At the start: 12 parts, among them J17 Pyro Terminal 1, J18 Pyro Terminal 2, Q4 AO4822A, U13 ILD213T

Commit message: v2!
Parts:
- C38, C39: value 100u -> 10u
- Q4: value AO4822A -> DMN3018SSD
